File: schematic/tinysynth.kicad_sch (KiCad schematic)
At the start: 11 parts, among them CN1 NMJ6HCD2, U1 ATtiny85-20S, U2 DIN-504D-M5

Commit message: did attiny25 socket version
Parts:
- removed U1: ATtiny85-20S, Package_SO:SOIC-8_5.3x5.3mm_P1.27mm, symbol MCU_Microchip_ATtiny:ATtiny85-20S
- added U1: ATtiny85-20P, Package_DIP:DIP-8_W7.62mm_Socket, symbol MCU_Microchip_ATtiny:ATtiny85-20P
Connections:
- net at C4.1, R1.2, U2.5: now also U1.5 (AREF/PB0)
- net at C1.2, C2.2, C3.2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: now also U1.4 (GND)
- net at C1.1, C2.1, R1.1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: now also U1.8 (VCC)
- net at R2.2: now also U1.6 (PB1)
